Commit message: controller suport

File: maze_runner_ws/src/maze_runner_description/urdf/maze_runner.urdf.xacro (robot description, xacro)
@@ -1,104 +1,5 @@
 <?xml version="1.0"?>
-<robot xmlns:xacro="http://www.ros.org/wiki/xacro" name="maze_runner">
-    <material name="blue"><color rgba="0.2 0.2 1.0 1.0"/></material>
-    <material name="black"><color rgba="0.1 0.1 0.1 1.0"/></material>
-    <material name="red"><color rgba="1.0 0.0 0.0 1.0"/></material>
-    <link name="base_footprint"/>
-    <joint name="base_joint" type="fixed">
-        <parent link="base_footprint"/>
-        <child link="base_link"/>
-        <origin xyz="0 0 0.1" rpy="0 0 0"/>
-    </joint>
-    <link name="base_link">
-        <visual>
-            <geometry><box size="0.4 0.3 0.15"/></geometry>
-            <material name="blue"/>
-        </visual>
-        <collision>
-            <geometry><box size="0.4 0.3 0.15"/></geometry>
-        </collision>
-        <inertial>
-            <mass value="5.0"/>
-            <inertia ixx="0.04" ixy="0.0" ixz="0.0" iyy="0.07" iyz="0.0" izz="0.1"/>
-        </inertial>
-    </link>
-    <joint name="caster_joint" type="fixed">
-        <parent link="base_link"/>
-        <child link="caster_link"/>
-        <origin xyz="-0.15 0 -0.075" rpy="0 0 0"/>
-    </joint>
-    <link name="caster_link">
-        <visual><geometry><sphere radius="0.025"/></geometry><material name="black"/></visual>
-        <collision><geometry><sphere radius="0.025"/></geometry></collision>
-        <surface><friction><ode><mu>0.0</mu><mu2>0.0</mu2></ode></friction></surface>
-        <inertial><mass value="0.5"/><inertia ixx="0.001" ixy="0.0" ixz="0.0" iyy="0.001" iyz="0.0" izz="0.001"/></inertial>
-    </link>
-    <joint name="left_wheel_joint" type="continuous">
-        <parent link="base_link"/>
-        <child link="left_wheel"/>
-        <origin xyz="0.1 0.175 -0.05" rpy="-1.5708 0 0"/> <axis xyz="0 0 1"/> </joint>
-    <link name="left_wheel">
-        <visual><geometry><cylinder radius="0.05" length="0.04"/></geometry><material name="black"/></visual>
-        <collision><geometry><cylinder radius="0.05" length="0.04"/></geometry></collision>
-        <inertial><mass value="1.0"/><inertia ixx="0.001" ixy="0.0" ixz="0.0" iyy="0.001" iyz="0.0" izz="0.001"/></inertial>
-    </link>
-    <joint name="right_wheel_joint" type="continuous">
-        <parent link="base_link"/>
-        <child link="right_wheel"/>
-        <origin xyz="0.1 -0.175 -0.05" rpy="-1.5708 0 0"/>
-        <axis xyz="0 0 1"/>
-    </joint>
-    <link name="right_wheel">
-        <visual><geometry><cylinder radius="0.05" length="0.04"/></geometry><material name="black"/></visual>
-        <collision><geometry><cylinder radius="0.05" length="0.04"/></geometry></collision>
-        <inertial><mass value="1.0"/><inertia ixx="0.001" ixy="0.0" ixz="0.0" iyy="0.001" iyz="0.0" izz="0.001"/></inertial>
-    </link>
-    <joint name="lidar_joint" type="fixed">
-        <parent link="base_link"/>
-        <child link="lidar_link"/>
-        <origin xyz="0 0 0.1" rpy="0 0 0"/> </joint>
-    <link name="lidar_link">
-        <visual><geometry><cylinder radius="0.04" length="0.05"/></geometry><material name="red"/></visual>
-        <collision><geometry><cylinder radius="0.04" length="0.05"/></geometry></collision>
-        <inertial><mass value="0.2"/><inertia ixx="0.0001" ixy="0.0" ixz="0.0" iyy="0.0001" iyz="0.0" izz="0.0001"/></inertial>
-    </link>
-    <gazebo>
-        <plugin filename="gz-sim-diff-drive-system" name="gz::sim::systems::DiffDrive">
-            <left_joint>left_wheel_joint</left_joint>
-            <right_joint>right_wheel_joint</right_joint>
-            <wheel_separation>0.35</wheel_separation>
-            <wheel_radius>0.05</wheel_radius>
-            <topic>cmd_vel</topic> </plugin>
-            <frame_id>odom</frame_id>
-            <child_frame_id>base_footprint</child_frame_id>
-    </gazebo>
-    <gazebo>
-        <plugin filename="gz-sim-joint-state-publisher-system" name="gz::sim::systems::JointStatePublisher">
-        </plugin>
-    </gazebo>
-    <gazebo reference="lidar_link">
-        <sensor name="lidar" type="gpu_lidar">
-            <topic>scan</topic>
-            <update_rate>10</update_rate>
-            <gz_frame_id>lidar_link</gz_frame_id>
-            <ray>
-                <scan>
-                    <horizontal>
-                        <samples>360</samples>
-                        <resolution>1</resolution>
-                        <min_angle>-3.14159</min_angle>
-                        <max_angle>3.14159</max_angle>
-                    </horizontal>
-                </scan>
-                <range>
-                    <min>0.15</min> <max>8.0</max>  </range>
-            </ray>
-            <always_on>1</always_on>
-            <visualize>true</visualize> </sensor>
-    </gazebo>
-    <gazebo>
-        <plugin filename="gz-sim-sensors-system" name="gz::sim::systems::Sensors">
-            <render_engine>ogre2</render_engine>
-        </plugin>
-    </gazebo>
+<robot name="maze_runner" xmlns:xacro="http://www.ros.org/wiki/xacro">
+    <xacro:include filename="maze_runner_base.xacro" />
+    <xacro:include filename="maze_runner_gazebo.xacro" />
 </robot>
